Commit message: update

File: phybot_c2/urdf/phybot_c2_base.urdf (robot description, URDF)
Before this commit: robot phybot_c2, 25 links, 24 joints
Links:
- link base_link: geometry collision mesh filename=package://phybot_c2/meshes/base_link.STL; visual mesh filename=package://phybot_c2/meshes/base_link.STL
- link left_ankle_pitch: geometry collision mesh filename=package://phybot_c2/meshes/left_ankle_pitch.STL; visual mesh filename=package://phybot_c2/meshes/left_ankle_pitch.STL
- link left_ankle_roll: geometry collision mesh filename=package://phybot_c2/meshes/left_ankle_roll.STL; visual mesh filename=package://phybot_c2/meshes/left_ankle_roll.STL
- link left_elbow_pitch: geometry collision mesh filename=package://phybot_c2/meshes/left_elbow_pitch.STL; visual mesh filename=package://phybot_c2/meshes/left_elbow_pitch.STL
- link left_hip_pitch: geometry collision mesh filename=package://phybot_c2/meshes/left_hip_pitch.STL; visual mesh filename=package://phybot_c2/meshes/left_hip_pitch.STL
- link left_hip_roll: geometry collision mesh filename=package://phybot_c2/meshes/left_hip_roll.STL; visual mesh filename=package://phybot_c2/meshes/left_hip_roll.STL
- link left_hip_yaw: geometry collision mesh filename=package://phybot_c2/meshes/left_hip_yaw.STL; visual mesh filename=package://phybot_c2/meshes/left_hip_yaw.STL
- link left_knee: geometry collision mesh filename=package://phybot_c2/meshes/left_knee.STL; visual mesh filename=package://phybot_c2/meshes/left_knee.STL
- link left_shoulder_pitch: geometry collision mesh filename=package://phybot_c2/meshes/left_shoulder_pitch.STL; visual mesh filename=package://phybot_c2/meshes/left_shoulder_pitch.STL
- link left_shoulder_roll: geometry collision mesh filename=package://phybot_c2/meshes/left_shoulder_roll.STL; visual mesh filename=package://phybot_c2/meshes/left_shoulder_roll.STL
- link left_shoulder_yaw: geometry collision mesh filename=package://phybot_c2/meshes/left_shoulder_yaw.STL; visual mesh filename=package://phybot_c2/meshes/left_shoulder_yaw.STL
- link neck_pitch: mass 0.05 -> 0.01; geometry collision mesh filename=package://phybot_c2/meshes/neck_pitch.STL; visual mesh filename=package://phybot_c2/meshes/neck_pitch.STL
- link neck_yaw: geometry collision mesh filename=package://phybot_c2/meshes/neck_yaw.STL; visual mesh filename=package://phybot_c2/meshes/neck_yaw.STL
- link right_ankle_pitch: geometry collision mesh filename=package://phybot_c2/meshes/right_ankle_pitch.STL; visual mesh filename=package://phybot_c2/meshes/right_ankle_pitch.STL
- link right_ankle_roll: geometry collision mesh filename=package://phybot_c2/meshes/right_ankle_roll.STL; visual mesh filename=package://phybot_c2/meshes/right_ankle_roll.STL
- link right_elbow_pitch: geometry collision mesh filename=package://phybot_c2/meshes/right_elbow_pitch.STL; visual mesh filename=package://phybot_c2/meshes/right_elbow_pitch.STL
- link right_hip_pitch: geometry collision mesh filename=package://phybot_c2/meshes/right_hip_pitch.STL; visual mesh filename=package://phybot_c2/meshes/right_hip_pitch.STL
- link right_hip_roll: geometry collision mesh filename=package://phybot_c2/meshes/right_hip_roll.STL; visual mesh filename=package://phybot_c2/meshes/right_hip_roll.STL
- link right_hip_yaw: geometry collision mesh filename=package://phybot_c2/meshes/right_hip_yaw.STL; visual mesh filename=package://phybot_c2/meshes/right_hip_yaw.STL
- link right_knee: geometry collision mesh filename=package://phybot_c2/meshes/right_knee.STL; visual mesh filename=package://phybot_c2/meshes/right_knee.STL
- link right_shoulder_pitch: geometry collision mesh filename=package://phybot_c2/meshes/right_shoulder_pitch.STL; visual mesh filename=package://phybot_c2/meshes/right_shoulder_pitch.STL
- link right_shoulder_roll: geometry collision mesh filename=package://phybot_c2/meshes/right_shoulder_roll.STL; visual mesh filename=package://phybot_c2/meshes/right_shoulder_roll.STL
- link right_shoulder_yaw: geometry collision mesh filename=package://phybot_c2/meshes/right_shoulder_yaw.STL; visual mesh filename=package://phybot_c2/meshes/right_shoulder_yaw.STL
- link torso: geometry collision mesh filename=package://phybot_c2/meshes/torso.STL; visual mesh filename=package://phybot_c2/meshes/torso.STL
- link waist_yaw: geometry collision mesh filename=package://phybot_c2/meshes/waist_yaw.STL; visual mesh filename=package://phybot_c2/meshes/waist_yaw.STL
Joints:
- joint left_ankle_pitch: limit lower=-1.57 upper=1.57 effort=58 velocity=98.37 -> lower=-1.57 upper=1.57 effort=58 velocity=8.37
- joint left_ankle_roll: limit lower=-1.13 upper=1.13 effort=58 velocity=98.37 -> lower=-1.13 upper=1.13 effort=58 velocity=8.37
- joint left_elbow_pitch: limit lower=-2.36 upper=0 effort=9 velocity=98.16 -> lower=-2.36 upper=0 effort=9 velocity=8.16
- joint left_hip_pitch: limit lower=-3.05 upper=2.09 effort=200 velocity=99.21 -> lower=-3.05 upper=2.09 effort=200 velocity=9.21
- joint left_hip_roll: limit lower=-0.44 upper=3.05 effort=80 velocity=98.9 -> lower=-0.44 upper=3.05 effort=80 velocity=8.9
- joint left_hip_yaw: limit lower=-2.53 upper=2.53 effort=58 velocity=98.37 -> lower=-2.53 upper=2.53 effort=58 velocity=8.37
- joint left_knee: limit lower=-0.05 upper=2.36 effort=80 velocity=98.9 -> lower=-0.05 upper=2.36 effort=80 velocity=8.9
- joint left_shoulder_pitch: limit lower=-3.58 upper=2.01 effort=58 velocity=98.37 -> lower=-3.58 upper=2.01 effort=58 velocity=8.37
- joint left_shoulder_roll: limit lower=-0.35 upper=3.05 effort=58 velocity=98.37 -> lower=-0.35 upper=3.05 effort=58 velocity=8.37
- joint left_shoulder_yaw: limit lower=-2.53 upper=2.53 effort=58 velocity=98.37 -> lower=-2.53 upper=2.53 effort=58 velocity=8.37
- joint neck_pitch: limit lower=-0.61 upper=0.61 effort=9 velocity=98.16 -> lower=-0.61 upper=0.61 effort=9 velocity=8.16; type fixed -> revolute
- joint neck_yaw: limit lower=-2.62 upper=2.62 effort=9 velocity=98.16 -> lower=-2.62 upper=2.62 effort=9 velocity=8.16; type fixed -> revolute
- joint right_ankle_pitch: limit lower=-1.57 upper=1.57 effort=58 velocity=98.37 -> lower=-1.57 upper=1.57 effort=58 velocity=8.37
- joint right_ankle_roll: limit lower=-1.13 upper=1.13 effort=58 velocity=98.37 -> lower=-1.13 upper=1.13 effort=58 velocity=8.37
- joint right_elbow_pitch: limit lower=-2.36 upper=0 effort=58 velocity=98.37 -> lower=-2.36 upper=0 effort=58 velocity=8.37
- joint right_hip_pitch: limit lower=-3.05 upper=2.09 effort=200 velocity=99.21 -> lower=-3.05 upper=2.09 effort=200 velocity=9.21
- joint right_hip_roll: limit lower=-3.05 upper=0.44 effort=80 velocity=98.9 -> lower=-3.05 upper=0.44 effort=80 velocity=8.9
- joint right_hip_yaw: limit lower=-2.53 upper=2.53 effort=58 velocity=98.37 -> lower=-2.53 upper=2.53 effort=58 velocity=8.37
- joint right_knee: limit lower=-0.05 upper=2.36 effort=80 velocity=98.9 -> lower=-0.05 upper=2.36 effort=80 velocity=8.9
- joint right_shoulder_pitch: limit lower=-3.58 upper=2.01 effort=58 velocity=98.37 -> lower=-3.58 upper=2.01 effort=58 velocity=8.37
- joint right_shoulder_roll: limit lower=-3.05 upper=0.35 effort=58 velocity=98.37 -> lower=-3.05 upper=0.35 effort=58 velocity=8.37
- joint right_shoulder_yaw: limit lower=-2.53 upper=2.53 effort=58 velocity=98.37 -> lower=-2.53 upper=2.53 effort=58 velocity=8.37
- joint waist_yaw: limit lower=-2.62 upper=2.62 effort=58 velocity=98.37 -> lower=-2.62 upper=2.62 effort=58 velocity=8.37

File: phybot_c2/urdf/phybot_c2_s_34.urdf (robot description, URDF)
Before this commit: robot phybot_c2, 25 links, 24 joints
Links:
- added link left_toe, mass 0.1; visual sphere radius=0.01
- added link right_toe, mass 0.1; visual sphere radius=0.01
- link base_link: mass 3.2436 -> 3.7383; geometry collision sphere radius=0.07; visual mesh filename=../new_meshes/base_link.STL
- link left_ankle_pitch: mass 1.55163108561377 -> 1.53; geometry collision sphere radius=0.045; visual mesh filename=../new_meshes/left_ankle_pitch.STL
- link left_ankle_roll: mass 0.388009531160459 -> 1.04; geometry collision cylinder length=0.24 radius=0.012; collision cylinder length=0.24 radius=0.012
- link left_elbow_pitch: mass 0.851991701787346 -> 1.84; geometry collision cylinder length=0.22 radius=0.035; visual mesh filename=../new_meshes/left_elbow_pitch.STL
- link left_hip_pitch: mass 0.91042 -> 1.0909; geometry visual mesh filename=../new_meshes/left_hip_pitch.STL
- link left_hip_roll: mass 0.23681 -> 0.2618; geometry collision sphere radius=0.05; visual mesh filename=../new_meshes/left_hip_roll.STL
- link left_hip_yaw: mass 1.00442326218312 -> 1.5; geometry collision cylinder length=0.18 radius=0.04; visual mesh filename=../new_meshes/left_hip_yaw.STL
- link left_knee: mass 1.35068107452534 -> 1.75; geometry collision cylinder length=0.16 radius=0.04; visual mesh filename=../new_meshes/left_knee.STL
- link left_shoulder_pitch: geometry visual mesh filename=../new_meshes/left_shoulder_pitch.STL
- link left_shoulder_roll: mass 0.224784045580485 -> 0.239; geometry collision sphere radius=0.05; visual mesh filename=../new_meshes/left_shoulder_roll.STL
- link left_shoulder_yaw: mass 1.59289091864703 -> 1.1136; geometry collision cylinder length=0.14 radius=0.03; visual mesh filename=../new_meshes/left_shoulder_yaw.STL
- link neck_pitch: mass 0.05 -> 2.36; geometry collision sphere radius=0.07; visual mesh filename=../new_meshes/neck_pitch.STL
- link neck_yaw: geometry visual mesh filename=../new_meshes/neck_yaw.STL
- link right_ankle_pitch: geometry collision sphere radius=0.045; visual mesh filename=../new_meshes/right_ankle_pitch.STL
- link right_ankle_roll: mass 0.397122220931611 -> 1.04; geometry collision cylinder length=0.24 radius=0.012; collision cylinder length=0.24 radius=0.012
- link right_elbow_pitch: mass 0.852091777096898 -> 1.84; geometry collision cylinder length=0.22 radius=0.035; visual mesh filename=../new_meshes/right_elbow_pitch.STL
- link right_hip_pitch: mass 0.910416842241314 -> 1.0909; geometry visual mesh filename=../new_meshes/right_hip_pitch.STL
- link right_hip_roll: mass 0.236808848887827 -> 0.2618; geometry collision sphere radius=0.05; visual mesh filename=../new_meshes/right_hip_roll.STL
- link right_hip_yaw: mass 1.0044272654158 -> 1.5; geometry collision cylinder length=0.18 radius=0.04; visual mesh filename=../new_meshes/right_hip_yaw.STL
- link right_knee: mass 1.35067962196111 -> 1.75; geometry collision cylinder length=0.16 radius=0.04; visual mesh filename=../new_meshes/right_knee.STL
- link right_shoulder_pitch: geometry visual mesh filename=../new_meshes/right_shoulder_pitch.STL
- link right_shoulder_roll: mass 0.224782671869933 -> 0.239; geometry collision sphere radius=0.05; visual mesh filename=../new_meshes/right_shoulder_roll.STL
- link right_shoulder_yaw: mass 1.59289091833568 -> 1.1136; geometry collision cylinder length=0.14 radius=0.03; visual mesh filename=../new_meshes/right_shoulder_yaw.STL
- link torso: mass 7.89499645954187 -> 7.4132; geometry collision box size=0.14 0.18 0.28; visual mesh filename=../new_meshes/torso.STL
- link waist_yaw: geometry visual mesh filename=../new_meshes/waist_yaw.STL
Joints:
- added joint left_toe: type fixed, parent left_ankle_roll, child left_toe, origin xyz=0.0875 0 -0.014 rpy=0 0 0
- added joint right_toe: type fixed, parent right_ankle_roll, child right_toe, origin xyz=0.0875 0 -0.014 rpy=0 0 0
- joint left_elbow_pitch: limit lower=-2.36 upper=0 effort=9 velocity=98.16 -> lower=-2.36 upper=0 effort=58 velocity=98.16

File: phybot_c2/urdf/phybot_c2_s_half.urdf (robot description, URDF)
Before this commit: robot phybot_c2, 25 links, 24 joints
Links:
- added link left_toe, mass 0.1; visual sphere radius=0.01
- added link right_toe, mass 0.1; visual sphere radius=0.01
- link base_link: mass 3.2436 -> 3.7383; geometry collision sphere radius=0.07; visual mesh filename=../new_meshes/base_link.STL
- link left_ankle_pitch: mass 1.55163108561377 -> 1.53; geometry collision sphere radius=0.045; visual mesh filename=../new_meshes/left_ankle_pitch.STL
- link left_ankle_roll: mass 0.388009531160459 -> 1.04; geometry collision cylinder length=0.24 radius=0.012; collision cylinder length=0.24 radius=0.012
- link left_elbow_pitch: mass 0.851991701787346 -> 1.84; geometry collision cylinder length=0.22 radius=0.035; visual mesh filename=../new_meshes/left_elbow_pitch.STL
- link left_hip_pitch: mass 0.91042 -> 1.0909; geometry visual mesh filename=../new_meshes/left_hip_pitch.STL
- link left_hip_roll: mass 0.23681 -> 0.2618; geometry collision sphere radius=0.05; visual mesh filename=../new_meshes/left_hip_roll.STL
- link left_hip_yaw: mass 1.00442326218312 -> 1.5; geometry collision cylinder length=0.18 radius=0.04; visual mesh filename=../new_meshes/left_hip_yaw.STL
- link left_knee: mass 1.35068107452534 -> 1.75; geometry collision cylinder length=0.16 radius=0.04; visual mesh filename=../new_meshes/left_knee.STL
- link left_shoulder_pitch: geometry visual mesh filename=../new_meshes/left_shoulder_pitch.STL
- link left_shoulder_roll: mass 0.224784045580485 -> 0.239; geometry collision sphere radius=0.05; visual mesh filename=../new_meshes/left_shoulder_roll.STL
- link left_shoulder_yaw: mass 1.59289091864703 -> 1.1136; geometry collision cylinder length=0.14 radius=0.03; visual mesh filename=../new_meshes/left_shoulder_yaw.STL
- link neck_pitch: mass 0.05 -> 2.36; geometry collision sphere radius=0.07; visual mesh filename=../new_meshes/neck_pitch.STL
- link neck_yaw: geometry visual mesh filename=../new_meshes/neck_yaw.STL
- link right_ankle_pitch: geometry collision sphere radius=0.045; visual mesh filename=../new_meshes/right_ankle_pitch.STL
- link right_ankle_roll: mass 0.397122220931611 -> 1.04; geometry collision cylinder length=0.24 radius=0.012; collision cylinder length=0.24 radius=0.012
- link right_elbow_pitch: mass 0.852091777096898 -> 1.84; geometry collision cylinder length=0.22 radius=0.035; visual mesh filename=../new_meshes/right_elbow_pitch.STL
- link right_hip_pitch: mass 0.910416842241314 -> 1.0909; geometry visual mesh filename=../new_meshes/right_hip_pitch.STL
- link right_hip_roll: mass 0.236808848887827 -> 0.2618; geometry collision sphere radius=0.05; visual mesh filename=../new_meshes/right_hip_roll.STL
- link right_hip_yaw: mass 1.0044272654158 -> 1.5; geometry collision cylinder length=0.18 radius=0.04; visual mesh filename=../new_meshes/right_hip_yaw.STL
- link right_knee: mass 1.35067962196111 -> 1.75; geometry collision cylinder length=0.16 radius=0.04; visual mesh filename=../new_meshes/right_knee.STL
- link right_shoulder_pitch: geometry visual mesh filename=../new_meshes/right_shoulder_pitch.STL
- link right_shoulder_roll: mass 0.224782671869933 -> 0.239; geometry collision sphere radius=0.05; visual mesh filename=../new_meshes/right_shoulder_roll.STL
- link right_shoulder_yaw: mass 1.59289091833568 -> 1.1136; geometry collision cylinder length=0.14 radius=0.03; visual mesh filename=../new_meshes/right_shoulder_yaw.STL
- link torso: mass 7.89499645954187 -> 7.4132; geometry collision box size=0.14 0.18 0.28; visual mesh filename=../new_meshes/torso.STL
- link waist_yaw: geometry visual mesh filename=../new_meshes/waist_yaw.STL
Joints:
- added joint left_toe: type fixed, parent left_ankle_roll, child left_toe, origin xyz=0.0875 0 -0.014 rpy=0 0 0
- added joint right_toe: type fixed, parent right_ankle_roll, child right_toe, origin xyz=0.0875 0 -0.014 rpy=0 0 0
- joint left_elbow_pitch: type revolute -> fixed
- joint left_shoulder_pitch: type revolute -> fixed
- joint left_shoulder_roll: type revolute -> fixed
- joint left_shoulder_yaw: type revolute -> fixed
- joint right_elbow_pitch: type revolute -> fixed
- joint right_shoulder_pitch: type revolute -> fixed
- joint right_shoulder_roll: type revolute -> fixed
- joint right_shoulder_yaw: type revolute -> fixed
