Commit message: update c2 model

File: phybot_c2/urdf/phybot_c2.urdf (robot description, URDF)
Before this commit: robot phybot_c2, 25 links, 24 joints
Links:
- added link left_wrist_yaw; visual sphere radius=0.05
- added link right_wrist_yaw; visual sphere radius=0.05
- link base_link: mass 3.2436 -> 7.2436; geometry collision sphere radius=0.07; visual mesh filename=../meshes/base_link.STL
- link left_ankle_pitch: geometry collision sphere radius=0.045; visual mesh filename=../meshes/left_ankle_pitch.STL
- link left_ankle_roll: geometry collision cylinder length=0.15 radius=0.01; collision cylinder length=0.15 radius=0.01
- link left_elbow_pitch: geometry collision cylinder length=0.22 radius=0.035; visual mesh filename=../meshes/left_elbow_pitch.STL
- link left_hip_pitch: geometry visual mesh filename=../meshes/left_hip_pitch.STL
- link left_hip_roll: geometry collision sphere radius=0.05; visual mesh filename=../meshes/left_hip_roll.STL
- link left_hip_yaw: geometry collision cylinder length=0.18 radius=0.04; visual mesh filename=../meshes/left_hip_yaw.STL
- link left_knee: geometry collision cylinder length=0.16 radius=0.04; visual mesh filename=../meshes/left_knee.STL
- link left_shoulder_pitch: geometry visual mesh filename=../meshes/left_shoulder_pitch.STL
- link left_shoulder_roll: geometry collision sphere radius=0.05; visual mesh filename=../meshes/left_shoulder_roll.STL
- link left_shoulder_yaw: geometry collision cylinder length=0.14 radius=0.03; visual mesh filename=../meshes/left_shoulder_yaw.STL
- link neck_pitch: geometry collision sphere radius=0.07; visual mesh filename=../meshes/neck_pitch.STL
- link neck_yaw: geometry visual mesh filename=../meshes/neck_yaw.STL
- link right_ankle_pitch: geometry collision sphere radius=0.045; visual mesh filename=../meshes/right_ankle_pitch.STL
- link right_ankle_roll: geometry collision cylinder length=0.15 radius=0.01; collision cylinder length=0.15 radius=0.01
- link right_elbow_pitch: geometry collision cylinder length=0.22 radius=0.035; visual mesh filename=../meshes/right_elbow_pitch.STL
- link right_hip_pitch: geometry visual mesh filename=../meshes/right_hip_pitch.STL
- link right_hip_roll: geometry collision sphere radius=0.05; visual mesh filename=../meshes/right_hip_roll.STL
- link right_hip_yaw: geometry collision cylinder length=0.18 radius=0.04; visual mesh filename=../meshes/right_hip_yaw.STL
- link right_knee: geometry collision cylinder length=0.16 radius=0.04; visual mesh filename=../meshes/right_knee.STL
- link right_shoulder_pitch: geometry visual mesh filename=../meshes/right_shoulder_pitch.STL
- link right_shoulder_roll: geometry collision sphere radius=0.05; visual mesh filename=../meshes/right_shoulder_roll.STL
- link right_shoulder_yaw: geometry collision cylinder length=0.14 radius=0.03; visual mesh filename=../meshes/right_shoulder_yaw.STL
- link torso: mass 7.89499645954187 -> 11.89499645954187; geometry collision box size=0.14 0.18 0.28; visual mesh filename=../meshes/torso.STL
- link waist_yaw: geometry visual mesh filename=../meshes/waist_yaw.STL
Joints:
- added joint left_wrist_yaw: type fixed, parent left_elbow_pitch, child left_wrist_yaw, origin xyz=0 0 -0.27 rpy=0 0 0
- added joint right_wrist_yaw: type fixed, parent right_elbow_pitch, child right_wrist_yaw, origin xyz=0 0 -0.27 rpy=0 0 0
- joint left_ankle_pitch: limit lower=-1.57 upper=1.57 effort=58 velocity=98.37 -> lower=-1.57 upper=1.57 effort=90 velocity=98.37
- joint left_ankle_roll: limit lower=-1.13 upper=1.13 effort=58 velocity=98.37 -> lower=-1.13 upper=1.13 effort=90 velocity=98.37
- joint left_elbow_pitch: limit lower=-2.36 upper=0 effort=9 velocity=98.16 -> lower=-2.36 upper=0 effort=90 velocity=98.16
- joint left_hip_pitch: limit lower=-3.05 upper=2.09 effort=200 velocity=99.21 -> lower=-3.05 upper=2.09 effort=160 velocity=99.21
- joint left_hip_roll: limit lower=-0.44 upper=3.05 effort=80 velocity=98.9 -> lower=-0.44 upper=3.05 effort=100 velocity=98.9
- joint left_hip_yaw: limit lower=-2.53 upper=2.53 effort=58 velocity=98.37 -> lower=-2.53 upper=2.53 effort=90 velocity=98.37
- joint left_knee: limit lower=-0.05 upper=2.36 effort=80 velocity=98.9 -> lower=-0.05 upper=2.36 effort=100 velocity=98.9
- joint left_shoulder_pitch: limit lower=-3.58 upper=2.01 effort=58 velocity=98.37 -> lower=-3.14 upper=3.14 effort=90 velocity=98.37
- joint left_shoulder_roll: limit lower=-0.35 upper=3.05 effort=58 velocity=98.37 -> lower=-3.14 upper=3.14 effort=90 velocity=98.37
- joint left_shoulder_yaw: limit lower=-2.53 upper=2.53 effort=58 velocity=98.37 -> lower=-3.14 upper=3.14 effort=90 velocity=98.37
- joint neck_pitch: limit lower=-0.61 upper=0.61 effort=9 velocity=98.16 -> lower=-0.61 upper=0.61 effort=30 velocity=98.16
- joint neck_yaw: limit lower=-2.62 upper=2.62 effort=9 velocity=98.16 -> lower=-2.62 upper=2.62 effort=30 velocity=98.16
- joint right_ankle_pitch: limit lower=-1.57 upper=1.57 effort=58 velocity=98.37 -> lower=-1.57 upper=1.57 effort=90 velocity=98.37
- joint right_ankle_roll: limit lower=-1.13 upper=1.13 effort=58 velocity=98.37 -> lower=-1.13 upper=1.13 effort=90 velocity=98.37
- joint right_elbow_pitch: limit lower=-2.36 upper=0 effort=58 velocity=98.37 -> lower=-2.36 upper=0 effort=90 velocity=98.37
- joint right_hip_pitch: limit lower=-3.05 upper=2.09 effort=200 velocity=99.21 -> lower=-3.05 upper=2.09 effort=160 velocity=99.21
- joint right_hip_roll: limit lower=-3.05 upper=0.44 effort=80 velocity=98.9 -> lower=-3.05 upper=0.44 effort=100 velocity=98.9
- joint right_hip_yaw: limit lower=-2.53 upper=2.53 effort=58 velocity=98.37 -> lower=-2.53 upper=2.53 effort=90 velocity=98.37
- joint right_knee: limit lower=-0.05 upper=2.36 effort=80 velocity=98.9 -> lower=-0.05 upper=2.36 effort=100 velocity=98.9
- joint right_shoulder_pitch: limit lower=-3.58 upper=2.01 effort=58 velocity=98.37 -> lower=-3.14 upper=3.14 effort=90 velocity=98.37
- joint right_shoulder_roll: limit lower=-3.05 upper=0.35 effort=58 velocity=98.37 -> lower=-3.14 upper=3.14 effort=90 velocity=98.37
- joint right_shoulder_yaw: limit lower=-2.53 upper=2.53 effort=58 velocity=98.37 -> lower=-3.14 upper=3.14 effort=90 velocity=98.37
- joint waist_yaw: limit lower=-2.62 upper=2.62 effort=58 velocity=98.37 -> lower=-2.62 upper=2.62 effort=90 velocity=98.37
