Commit message: update

File: phybot_racing_v2/urdf/phybot_racing_v2.urdf (robot description, URDF)
Before this commit: robot phybot_racing_v2, 21 links, 20 joints
Links:
- added link world
Joints:
- added joint floating_base_joint: type floating, parent world, child base_link, origin xyz=0 0 0 rpy=0 0 0
