Commit message: update m1 model

File: phybot_big_v2/urdf/phybot_big_v2_24dof.urdf (robot description, URDF)
Before this commit: robot phybot_big_v2, 30 links, 29 joints
Links:
- link left_ankle_roll: geometry collision cylinder length=0.24 radius=0.015; collision cylinder length=0.24 radius=0.015
- link left_elbow_yaw: geometry collision cylinder length=0.05 radius=0.03; visual mesh filename=../meshes/left_elbow_yaw.STL
- link right_ankle_roll: geometry collision cylinder length=0.24 radius=0.015; collision cylinder length=0.254 radius=0.015
- link right_elbow_yaw: geometry collision cylinder length=0.05 radius=0.03; visual mesh filename=../meshes/right_elbow_yaw.STL
Joints:
- joint left_ankle_pitch: limit lower=-0.87 upper=0.52 effort=200 velocity=98.79 -> lower=-0.87 upper=0.52 effort=250 velocity=22
- joint left_ankle_roll: limit lower=-0.61 upper=0.61 effort=60 velocity=912.56 -> lower=-0.61 upper=0.61 effort=89 velocity=25
- joint left_elbow_pitch: limit lower=-2.36 upper=0 effort=58 velocity=8.16 -> lower=-2.36 upper=0 effort=89 velocity=25
- joint left_elbow_yaw: limit lower=-1.57 upper=1.57 effort=58 velocity=8.16 -> lower=-1.57 upper=1.57 effort=89 velocity=25; type fixed -> revolute
- joint left_hip_pitch: limit lower=-2.62 upper=2.62 effort=500 velocity=99.21 -> lower=-2.62 upper=2.62 effort=600 velocity=18
- joint left_hip_roll: limit lower=-0.17 upper=1.92 effort=200 velocity=98.9 -> lower=-0.17 upper=1.92 effort=200 velocity=22
- joint left_hip_yaw: limit lower=-1.57 upper=1.57 effort=200 velocity=98.37 -> lower=-1.57 upper=1.57 effort=250 velocity=22
- joint left_knee: limit lower=0 upper=2.62 effort=500 velocity=99.21 -> lower=0 upper=2.62 effort=600 velocity=18
- joint left_shoulder_pitch: limit lower=-2.79 upper=0.87 effort=200 velocity=8.9 -> lower=-2.79 upper=0.87 effort=200 velocity=22
- joint left_shoulder_roll: limit lower=-0.17 upper=3.14 effort=200 velocity=8.9 -> lower=-0.34 upper=3.14 effort=135 velocity=25
- joint left_shoulder_yaw: limit lower=-1.57 upper=1.57 effort=58 velocity=8.16 -> lower=-1.57 upper=1.57 effort=89 velocity=25
- joint right_ankle_pitch: limit lower=-0.87 upper=0.52 effort=200 velocity=98.79 -> lower=-0.87 upper=0.52 effort=250 velocity=22
- joint right_ankle_roll: limit lower=-0.61 upper=0.61 effort=60 velocity=912.56 -> lower=-0.61 upper=0.61 effort=89 velocity=25
- joint right_elbow_pitch: limit lower=-2.36 upper=0 effort=58 velocity=8.16 -> lower=-2.36 upper=0 effort=89 velocity=25
- joint right_elbow_yaw: limit lower=-1.57 upper=1.57 effort=58 velocity=8.16 -> lower=-1.57 upper=1.57 effort=89 velocity=25; type fixed -> revolute
- joint right_hip_pitch: limit lower=-2.62 upper=2.62 effort=500 velocity=99.21 -> lower=-2.62 upper=2.62 effort=600 velocity=18
- joint right_hip_roll: limit lower=-1.92 upper=0.17 effort=200 velocity=98.9 -> lower=-1.92 upper=0.17 effort=200 velocity=22
- joint right_hip_yaw: limit lower=-1.57 upper=1.57 effort=200 velocity=98.37 -> lower=-1.57 upper=1.57 effort=250 velocity=22
- joint right_knee: limit lower=0 upper=2.62 effort=500 velocity=99.21 -> lower=0 upper=2.62 effort=600 velocity=18
- joint right_shoulder_pitch: limit lower=-2.79 upper=0.87 effort=200 velocity=8.9 -> lower=-2.79 upper=0.87 effort=200 velocity=22
- joint right_shoulder_roll: limit lower=-3.14 upper=0.17 effort=200 velocity=8.9 -> lower=-3.14 upper=0.34 effort=135 velocity=25
- joint right_shoulder_yaw: limit lower=-1.57 upper=1.57 effort=58 velocity=8.16 -> lower=-1.57 upper=1.57 effort=89 velocity=25
- joint waist_roll: limit lower=-0.79 upper=0.79 effort=200 velocity=98.9 -> lower=-0.79 upper=0.79 effort=200 velocity=22
- joint waist_yaw: limit lower=-1.57 upper=1.57 effort=230 velocity=98.37 -> lower=-1.57 upper=1.57 effort=250 velocity=22
